File: CMU Roboclub dGPS/dGPS_mainBoard.sch (EAGLE design)
At the start: 14 parts, among them IC1 LM2937

Commit message: Changed several things
Parts:
- removed U$2: VENUS822A, skytraq:VENUS822A
- added S5: Mode Sel., switch:320-938
- added SV1: FTDI, con-lstb:MA06-1
- S1: value Mode Select -> xBee RST; device switch:316-923 -> switch:TL32YO
- S2: value USB Data -> PWR SEL; device switch:316-923 -> switch:TL36PO
- S3: value xBee Data -> FTDI Data; device switch:316-923 -> switch:320-938
- S4: value TL32WO -> xBee Data; device switch:TL32WO -> switch:320-938
Connections:
- new net N$15: C1.1, IC1.VI, S2.P
- new net N$16: S2.S, SV1.3
- net N$10: now also S4B.P; no longer S3B.P
- net N$11: now also S41.P; no longer S32.P
- net N$12: now also S1.S, SV1.1; no longer S4.S, U$2.GND
- net N$13: now also S1.P; no longer S4.P
- net N$14: now also S2.O; no longer C1.1, IC1.VI
- net N$2: now also S3B.P, SV1.5; no longer S2B.P, U$2.TXD
- net N$3: now also S5B.P; no longer S1B.P
- net N$4: now also S31.O; no longer S22.O
- net N$5: now also S41.O, S5B.O; no longer S1B.O, S32.O
- net N$6: now also S4B.O, S51.S; no longer S12.S, S3B.O
- net N$7: now also S51.O; no longer S12.O
- net N$8: now also S31.P, SV1.4; no longer S22.P, U$2.RXD
- net N$9: now also S3B.O, S51.P; no longer S12.P, S2B.O
Other:
- note added: "EXT"
- note added: "FTDI"
- note removed: "MODE SELECT"
- note removed: "RADIO DATA"
- note removed: "USB DATA"
- note removed: "XBEE RESET"
- moved on the sheet: C1, C2, C3, IC1, J1, NEMA, S3

Commit message: Added indicator LEDs and did other stuff
Parts:
- removed IC1: LM2937, linear:LM2937
- removed J1: (no value), con-jack:DCJ0303
- added LED1: PWR, SRG:JST-PH_2-PIN_HEADER
- added LED2: xBee Assoc., SRG:JST-PH_2-PIN_HEADER
- added LED3: xBee RX, SRG:JST-PH_2-PIN_HEADER
- added LED4: xBee TX, SRG:JST-PH_2-PIN_HEADER
- added LED5: xBee RX Strength, SRG:JST-PH_2-PIN_HEADER
- added PWR: JST-PH_2-PIN_HEADER, SRG:JST-PH_2-PIN_HEADER
- added R1, R2, R3, R4, R5: 1k, rcl:R-US_0204/5
- added U$2: LD1117V33, LD1117V33:LD1117V33
Connections:
- new net N$17: C1.2, C2.2, C3.2, C4.1, LED1.2, LED2.2, LED3.2, LED4.2, LED5.2, NEMA.2, PWR.2, S1.S, SV1.1, U$1.GND@1, U$1.RFGND@1, U$2.GND, XB1.GND
- new net N$18: R5.1, XB1.RSSI/PWM/DIO10
- new net N$19: LED1.1, R1.2
- new net N$20: LED2.1, R2.2
- new net N$21: LED3.1, R3.2
- new net N$22: LED4.1, R4.2
- new net N$23: LED5.1, R5.2
- net N$1: now also R1.1, U$2.OUT; no longer IC1.VO
- net N$10: now also R4.1
- net N$11: now also R3.1
- net N$12: now also R2.1, XB1.ASSOC/DIO5; no longer C1.2, C2.2, C3.2, C4.1, IC1.GND, J1.2, NEMA.2, S1.S, SV1.1, U$1.GND@1, U$1.RFGND@1, XB1.GND
- net N$14: now also PWR.1; no longer J1.1
- net N$15: now also U$2.IN; no longer IC1.VI
Other:
- moved on the sheet: C1, C2
